Commit message: Update navigasi

File: description/lidar.xacro (robot description, xacro)
@@ -1,8 +1,34 @@
 <?xml version="1.0"?>
 <robot xmlns:xacro="http://www.ros.org/wiki/xacro" >
+    <joint name="lidar_connector_joint" type="fixed">
+        <parent link="chassis"/>
+        <child link="lidar_connector"/>
+        <origin xyz="0 0 0.7" rpy="0 0 0" />
+    </joint>
+    <link name="lidar_connector">
+        <visual>
+            <origin xyz="0 0 0"/>
+            <geometry>
+                <box size="0.05 0.05 1.0"/>
+            </geometry>
+            <material name="orange"/>
+        </visual>
+        <collision>
+            <origin xyz="0 0 0"/>
+            <geometry>
+                <box size="0.05 0.05 1.0"/>
+            </geometry>
+        </collision>
+        <xacro:inertial_box mass="0.001" x="0.05" y="0.05" z="1.0">
+            <origin xyz="0 0 0" rpy="0 0 0"/>
+        </xacro:inertial_box>
+    </link>
+    <gazebo reference="lidar_connector">
+        <material>Gazebo/Orange</material>
+    </gazebo>
     <joint name="laser_joint" type="fixed">
-        <parent link="chassis"/>
+        <parent link="lidar_connector"/>
         <child link="laser_frame"/>
-        <origin xyz="0 0 0.2" rpy="0 0 0"/>
+        <origin xyz="0 0 0.5" rpy="0 0 0"/>
         <!-- <origin xyz="0.1 0 0.175" rpy="0 0 0"/> -->
     </joint>
@@ -27,5 +53,5 @@
         <sensor name="laser" type="ray">
             <pose> 0 0 0 0 0 0 </pose>
-            <visualize>true</visualize>
+            <!-- <visualize>true</visualize> -->
             <update_rate>10</update_rate>
             <ray>

File: description/robot_core.xacro (robot description, xacro)
@@ -6,5 +6,5 @@
     <xacro:property name="chassis_mass" value="20.0"/>
     <xacro:property name="wheel_radius" value="0.125"/>
-    <xacro:property name="wheel_thickness" value="0.05"/>
+    <xacro:property name="wheel_thickness" value="0.04"/>
     <xacro:property name="wheel_mass" value="0.05"/>
     <xacro:property name="wheel_offset_x" value="0"/>
@@ -14,5 +14,5 @@
     <xacro:property name="caster_wheel_mass" value="0.01"/>
     <xacro:property name="connector_size" value="0.02"/>
-    <xacro:property name="connector_height" value="0.055"/>
+    <xacro:property name="connector_height" value="0.15"/>
     <xacro:property name="connector_offset_z" value="-0.02"/>
     <xacro:property name="caster_wheel_offset_x" value="0.1"/>

File: description/ultrasonic.xacro (robot description, xacro)
@@ -1,11 +1,14 @@
 <?xml version="1.0"?>
 <robot xmlns:xacro="http://www.ros.org/wiki/xacro">
-    <joint name="ultrasonic_sensor_joint" type="fixed">
-        <parent link="chassis"/>
-        <child link="ultrasonic_frame"/>
-        <origin xyz="${chassis_length/2} 0 ${chassis_height/2}" rpy="0 0 0"/>
-    </joint>
-    <link name="ultrasonic_frame">
-        <!-- Rectangular Base -->
+    <xacro:property name="us_offset_x" value="${chassis_length/2 + 0.003}"/>
+    <xacro:property name="us_offset_y" value="0.1"/>
+    <xacro:property name="us_offset_z" value="${chassis_height/2}"/>
+    <xacro:property name="us_rotation_yaw" value="0.55"/> <!-- 3.14rad = 180 degrees, 0.1rad = 5.7degrees -->
+    <joint name="fr_mid_us_joint" type="fixed">
+        <parent link="chassis"/>
+        <child link="fr_mid_us_frame"/>
+        <origin xyz="${us_offset_x} 0 ${us_offset_z}" rpy="0 0 0"/>
+    </joint>
+    <link name="fr_mid_us_frame">
         <visual>
             <geometry>
@@ -24,7 +27,7 @@
         </xacro:inertial_cylinder>
     </link>
-    <gazebo reference="ultrasonic_frame">
-        <material>Gazebo/Red</material>
-        <sensor type="ray" name="range_sensor">
+    <gazebo reference="fr_mid_us_frame">
+        <material>Gazebo/Red</material>
+        <sensor type="ray" name="fr_mid_range_sensor">
             <visualize>true</visualize>
             <pose> 0 0 0 0 0 0 </pose>
@@ -45,21 +48,192 @@
                 </scan>
                 <range>
-                    <min>0.10</min>
-                    <max>5.0</max>
-                    <resolution>0.01</resolution>
-                </range>
-                <noise>
-                    <type>gaussian</type>
-                    <mean>0.0</mean>
-                    <stddev>0.01</stddev>
-                </noise>
-            </ray>
-            <update_rate>30</update_rate>
-            <plugin name="gazebo_ros_range_controller" filename="libgazebo_ros_ray_sensor.so">
-                <ros>
-                    <remapping>~/out:=range</remapping>
-                </ros>
-                <output_type>sensor_msgs/Range</output_type>
-                <frame_name>ultrasonic_frame</frame_name>
+                    <min>0.2</min>
+                    <max>5.0</max>
+                    <resolution>0.01</resolution>
+                </range>
+                <noise>
+                    <type>gaussian</type>
+                    <mean>0.0</mean>
+                    <stddev>0.01</stddev>
+                </noise>
+            </ray>
+            <update_rate>30</update_rate>
+            <plugin name="fr_mid_us_controller" filename="libgazebo_ros_ray_sensor.so">
+                <ros>
+                    <remapping>~/out:=fr_mid_range</remapping>
+                </ros>
+                <output_type>sensor_msgs/Range</output_type>
+                <frame_name>fr_mid_us_frame</frame_name>
+            </plugin>
+        </sensor>
+    </gazebo>
+    <joint name="fr_left_us_joint" type="fixed">
+        <parent link="chassis"/>
+        <child link="fr_left_us_frame"/>
+        <origin xyz="${us_offset_x - 0.023} ${us_offset_y} ${us_offset_z}" rpy="0 0 ${us_rotation_yaw}"/>
+    </joint>
+    <link name="fr_left_us_frame">
+        <visual>
+            <geometry>
+                <box size="0.005 0.04 0.02"/>
+            </geometry>
+            <origin xyz="0 0 -0.0025" rpy="0 0 0"/>
+        </visual>
+        <collision>
+            <geometry>
+                <box size="0.005 0.04 0.02"/>
+            </geometry>
+            <origin xyz="0 0 -0.0025" rpy="0 0 0"/>
+        </collision>
+        <xacro:inertial_cylinder mass="0.1" length="0.02" radius="0.01">
+            <origin xyz="0 0 0" rpy="0 0 0"/>
+        </xacro:inertial_cylinder>
+    </link>
+    <gazebo reference="fr_left_us_frame">
+        <material>Gazebo/Red</material>
+        <sensor type="ray" name="fr_left_range_sensor">
+            <visualize>true</visualize>
+            <pose> 0 0 0 0 0 0 </pose>
+            <ray>
+                <scan>
+                    <horizontal>
+                        <samples>10</samples>
+                        <resolution>1</resolution>
+                        <min_angle>-0.087</min_angle>
+                        <max_angle>0.087</max_angle>
+                    </horizontal>
+                </scan>
+                <range>
+                    <min>0.2</min>
+                    <max>5.0</max>
+                    <resolution>0.01</resolution>
+                </range>
+                <noise>
+                    <type>gaussian</type>
+                    <mean>0.0</mean>
+                    <stddev>0.01</stddev>
+                </noise>
+            </ray>
+            <update_rate>30</update_rate>
+            <plugin name="fr_left_us_controller" filename="libgazebo_ros_ray_sensor.so">
+                <ros>
+                    <remapping>~/out:=fr_left_range</remapping>
+                </ros>
+                <output_type>sensor_msgs/Range</output_type>
+                <frame_name>fr_left_us_frame</frame_name>
+            </plugin>
+        </sensor>
+    </gazebo>
+    <joint name="fr_right_us_joint" type="fixed">
+        <parent link="chassis"/>
+        <child link="fr_right_us_frame"/>
+        <origin xyz="${us_offset_x - 0.023} ${-us_offset_y} ${us_offset_z}" rpy="0 0 ${-us_rotation_yaw}"/>
+    </joint>
+    <link name="fr_right_us_frame">
+        <visual>
+            <geometry>
+                <box size="0.005 0.04 0.02"/>
+            </geometry>
+            <origin xyz="0 0 -0.0025" rpy="0 0 0"/>
+        </visual>
+        <collision>
+            <geometry>
+                <box size="0.005 0.04 0.02"/>
+            </geometry>
+            <origin xyz="0 0 -0.0025" rpy="0 0 0"/>
+        </collision>
+        <xacro:inertial_cylinder mass="0.1" length="0.02" radius="0.01">
+            <origin xyz="0 0 0" rpy="0 0 0"/>
+        </xacro:inertial_cylinder>
+    </link>
+    <gazebo reference="fr_right_us_frame">
+        <material>Gazebo/Red</material>
+        <sensor type="ray" name="fr_right_range_sensor">
+            <visualize>true</visualize>
+            <pose> 0 0 0 0 0 0 </pose>
+            <ray>
+                <scan>
+                    <horizontal>
+                        <samples>10</samples>
+                        <resolution>1</resolution>
+                        <min_angle>-0.087</min_angle>
+                        <max_angle>0.087</max_angle>
+                    </horizontal>
+                </scan>
+                <range>
+                    <min>0.2</min>
+                    <max>5.0</max>
+                    <resolution>0.01</resolution>
+                </range>
+                <noise>
+                    <type>gaussian</type>
+                    <mean>0.0</mean>
+                    <stddev>0.01</stddev>
+                </noise>
+            </ray>
+            <update_rate>30</update_rate>
+            <plugin name="fr_right_us_controller" filename="libgazebo_ros_ray_sensor.so">
+                <ros>
+                    <remapping>~/out:=fr_right_range</remapping>
+                </ros>
+                <output_type>sensor_msgs/Range</output_type>
+                <frame_name>fr_right_us_frame</frame_name>
+            </plugin>
+        </sensor>
+    </gazebo>
+    <joint name="bc_mid_us_joint" type="fixed">
+        <parent link="chassis"/>
+        <child link="bc_mid_us_frame"/>
+        <origin xyz="${-us_offset_x} 0 ${us_offset_z}" rpy="0 0 3.14"/>
+    </joint>
+    <link name="bc_mid_us_frame">
+        <visual>
+            <geometry>
+                <box size="0.005 0.04 0.02"/>
+            </geometry>
+            <origin xyz="0 0 -0.0025" rpy="0 0 3.14"/>
+        </visual>
+        <collision>
+            <geometry>
+                <box size="0.005 0.04 0.02"/>
+            </geometry>
+            <origin xyz="0 0 -0.0025" rpy="0 0 3.14"/>
+        </collision>
+        <xacro:inertial_cylinder mass="0.1" length="0.02" radius="0.01">
+            <origin xyz="0 0 0" rpy="0 0 3.14"/>
+        </xacro:inertial_cylinder>
+    </link>
+    <gazebo reference="bc_mid_us_frame">
+        <material>Gazebo/Red</material>
+        <sensor type="ray" name="bc_mid_range_sensor">
+            <visualize>true</visualize>
+            <pose> 0 0 0 0 0 0 </pose>
+            <ray>
+                <scan>
+                    <horizontal>
+                        <samples>10</samples>
+                        <resolution>1</resolution>
+                        <min_angle>-0.087</min_angle>
+                        <max_angle>0.087</max_angle>
+                    </horizontal>
+                </scan>
+                <range>
+                    <min>0.2</min>
+                    <max>5.0</max>
+                    <resolution>0.01</resolution>
+                </range>
+                <noise>
+                    <type>gaussian</type>
+                    <mean>0.0</mean>
+                    <stddev>0.01</stddev>
+                </noise>
+            </ray>
+            <update_rate>30</update_rate>
+            <plugin name="bc_mid_us_controller" filename="libgazebo_ros_ray_sensor.so">
+                <ros>
+                    <remapping>~/out:=bc_mid_range</remapping>
+                </ros>
+                <output_type>sensor_msgs/Range</output_type>
+                <frame_name>bc_mid_us_frame</frame_name>
             </plugin>
         </sensor>
