Commit message: Update ultrasonic config

File: description/ultrasonic.xacro (robot description, xacro)
@@ -4,5 +4,5 @@
     <xacro:property name="us_offset_y" value="0.1"/>
     <xacro:property name="us_offset_z" value="${chassis_height/2}"/>
-    <xacro:property name="us_rotation_yaw" value="0.55"/> <!-- 3.14rad = 180 degrees, 0.1rad = 5.7degrees -->
+    <xacro:property name="us_rotation_yaw" value="0.25"/> <!-- 3.14rad = 180 degrees, 0.1rad = 5.7degrees -->
     <joint name="fr_mid_us_joint" type="fixed">
         <parent link="chassis"/>
@@ -49,5 +49,5 @@
                 <range>
                     <min>0.2</min>
-                    <max>5.0</max>
+                    <max>20</max>
                     <resolution>0.01</resolution>
                 </range>
@@ -114,5 +114,5 @@
                 <range>
                     <min>0.2</min>
-                    <max>5.0</max>
+                    <max>20</max>
                     <resolution>0.01</resolution>
                 </range>
@@ -179,5 +179,5 @@
                 <range>
                     <min>0.2</min>
-                    <max>5.0</max>
+                    <max>20</max>
                     <resolution>0.01</resolution>
                 </range>
@@ -244,5 +244,5 @@
                 <range>
                     <min>0.2</min>
-                    <max>5.0</max>
+                    <max>20</max>
                     <resolution>0.01</resolution>
                 </range>
