Commit message: Update ultrasonic description

File: description/gazebo_control.xacro (robot description, xacro)
@@ -7,7 +7,7 @@
             <right_joint>right_wheel_joint</right_joint>
             <wheel_separation>0.35</wheel_separation>
-            <wheel_diameter>0.1</wheel_diameter>
+            <wheel_diameter>0.125</wheel_diameter>
             <!-- Limits -->
-            <max_wheel_torque>200</max_wheel_torque>
+            <max_wheel_torque>1</max_wheel_torque>
             <max_wheel_acceleration>10.0</max_wheel_acceleration>
             <!-- Output -->

File: description/ultrasonic.xacro (robot description, xacro)
@@ -36,14 +36,14 @@
                     <horizontal>
                         <samples>10</samples>
-                        <resolution>1</resolution>
-                        <min_angle>-0.087</min_angle>
-                        <max_angle>0.087</max_angle>
-                    </horizontal>
-                    <!-- <vertical>
-                        <samples>10</samples>
-                        <resolution>1</resolution>
-                        <min_angle>-0.087</min_angle>
-                        <max_angle>0.087</max_angle>
-                    </vertical> -->
+                        <resolution>1.00000</resolution>
+                        <min_angle>-0.12</min_angle>
+                        <max_angle>0.12</max_angle>
+                    </horizontal>
+                    <vertical>
+                        <samples>1</samples>
+                        <resolution>1.00000</resolution>
+                        <min_angle>-0.01</min_angle>
+                        <max_angle>0.01</max_angle>
+                    </vertical>
                 </scan>
                 <range>
@@ -65,4 +65,6 @@
                 <output_type>sensor_msgs/Range</output_type>
                 <frame_name>fr_mid_us_frame</frame_name>
+                <field_of_view>0.01</field_of_view>
+                <radiation_type>ultrasound</radiation_type>
             </plugin>
         </sensor>
@@ -93,14 +95,20 @@
         <material>Gazebo/Red</material>
         <sensor type="ray" name="fr_left_range_sensor">
-            <visualize>true</visualize>
-            <pose> 0 0 0 0 0 0 </pose>
-            <ray>
-                <scan>
-                    <horizontal>
-                        <samples>10</samples>
-                        <resolution>1</resolution>
-                        <min_angle>-0.087</min_angle>
-                        <max_angle>0.087</max_angle>
-                    </horizontal>
+             <visualize>true</visualize>
+            <pose> 0 0 0 0 0 0 </pose>
+            <ray>
+                <scan>
+                    <horizontal>
+                        <samples>10</samples>
+                        <resolution>1.00000</resolution>
+                        <min_angle>-0.12</min_angle>
+                        <max_angle>0.12</max_angle>
+                    </horizontal>
+                    <vertical>
+                        <samples>1</samples>
+                        <resolution>1.00000</resolution>
+                        <min_angle>-0.01</min_angle>
+                        <max_angle>0.01</max_angle>
+                    </vertical>
                 </scan>
                 <range>
@@ -122,4 +130,6 @@
                 <output_type>sensor_msgs/Range</output_type>
                 <frame_name>fr_left_us_frame</frame_name>
+                <field_of_view>0.01</field_of_view>
+                <radiation_type>ultrasound</radiation_type>
             </plugin>
         </sensor>
@@ -150,14 +160,20 @@
         <material>Gazebo/Red</material>
         <sensor type="ray" name="fr_right_range_sensor">
-            <visualize>true</visualize>
-            <pose> 0 0 0 0 0 0 </pose>
-            <ray>
-                <scan>
-                    <horizontal>
-                        <samples>10</samples>
-                        <resolution>1</resolution>
-                        <min_angle>-0.087</min_angle>
-                        <max_angle>0.087</max_angle>
-                    </horizontal>
+             <visualize>true</visualize>
+            <pose> 0 0 0 0 0 0 </pose>
+            <ray>
+                <scan>
+                    <horizontal>
+                        <samples>10</samples>
+                        <resolution>1.00000</resolution>
+                        <min_angle>-0.12</min_angle>
+                        <max_angle>0.12</max_angle>
+                    </horizontal>
+                    <vertical>
+                        <samples>1</samples>
+                        <resolution>1.00000</resolution>
+                        <min_angle>-0.01</min_angle>
+                        <max_angle>0.01</max_angle>
+                    </vertical>
                 </scan>
                 <range>
@@ -179,4 +195,6 @@
                 <output_type>sensor_msgs/Range</output_type>
                 <frame_name>fr_right_us_frame</frame_name>
+                <field_of_view>0.01</field_of_view>
+                <radiation_type>ultrasound</radiation_type>
             </plugin>
         </sensor>
@@ -213,8 +231,14 @@
                     <horizontal>
                         <samples>10</samples>
-                        <resolution>1</resolution>
-                        <min_angle>-0.087</min_angle>
-                        <max_angle>0.087</max_angle>
-                    </horizontal>
+                        <resolution>1.00000</resolution>
+                        <min_angle>-0.12</min_angle>
+                        <max_angle>0.12</max_angle>
+                    </horizontal>
+                    <vertical>
+                        <samples>1</samples>
+                        <resolution>1.00000</resolution>
+                        <min_angle>-0.01</min_angle>
+                        <max_angle>0.01</max_angle>
+                    </vertical>
                 </scan>
                 <range>
@@ -236,4 +260,6 @@
                 <output_type>sensor_msgs/Range</output_type>
                 <frame_name>bc_mid_us_frame</frame_name>
+                <field_of_view>0.01</field_of_view>
+                <radiation_type>ultrasound</radiation_type>
             </plugin>
         </sensor>

File: description/ultrasonic_copy.xacro (robot description, xacro)
@@ -1,11 +1,14 @@
 <?xml version="1.0"?>
 <robot xmlns:xacro="http://www.ros.org/wiki/xacro">
-    <joint name="ultrasonic_sensor_joint" type="fixed">
-        <parent link="chassis"/>
-        <child link="ultrasonic_frame"/>
-        <origin xyz="${chassis_length/2} 0 ${chassis_height/2}" rpy="0 0 0"/>
-    </joint>
-    <link name="ultrasonic_frame">
-        <!-- Rectangular Base -->
+    <xacro:property name="us_offset_x" value="${chassis_length/2 + 0.003}"/>
+    <xacro:property name="us_offset_y" value="0.1"/>
+    <xacro:property name="us_offset_z" value="${chassis_height/2}"/>
+    <xacro:property name="us_rotation_yaw" value="0.55"/> <!-- 3.14rad = 180 degrees, 0.1rad = 5.7degrees -->
+    <joint name="fr_mid_us_joint" type="fixed">
+        <parent link="chassis"/>
+        <child link="fr_mid_us_frame"/>
+        <origin xyz="${us_offset_x} 0 ${us_offset_z}" rpy="0 0 0"/>
+    </joint>
+    <link name="fr_mid_us_frame">
         <visual>
             <geometry>
@@ -24,7 +27,67 @@
         </xacro:inertial_cylinder>
     </link>
-    <gazebo reference="ultrasonic_frame">
-        <material>Gazebo/Red</material>
-        <sensor type="ray" name="range_sensor">
+    <gazebo reference="fr_mid_us_frame">
+        <material>Gazebo/Red</material>
+        <sensor type="ray" name="fr_mid_range_sensor">
+            <visualize>true</visualize>
+            <pose> 0 0 0 0 0 0 </pose>
+            <ray>
+                <scan>
+                    <horizontal>
+                        <samples>10</samples>
+                        <resolution>1.00000</resolution>
+                        <min_angle>-0.12</min_angle>
+                        <max_angle>0.12</max_angle>
+                    </horizontal>
+                    <vertical>
+                        <samples>5</samples>
+                        <resolution>1.00000</resolution>
+                        <min_angle>-0.01</min_angle>
+                        <max_angle>0.01</max_angle>
+                    </vertical>
+                </scan>
+                <range>
+                    <min>0.2</min>
+                    <max>5.0</max>
+                    <resolution>0.01</resolution>
+                </range>
+            </ray>
+            <update_rate>20</update_rate>
+            <plugin name="fr_mid_us_controller" filename="libgazebo_ros_ray_sensor.so">
+                <ros>
+                    <remapping>~/out:=fr_mid_range</remapping>
+                </ros>
+                <output_type>sensor_msgs/Range</output_type>
+                <frame_name>fr_mid_us_frame</frame_name>
+                <field_of_view>0.01</field_of_view>
+                <radiation_type>ultrasound</radiation_type>
+            </plugin>
+        </sensor>
+    </gazebo>
+    <!-- <joint name="fr_left_us_joint" type="fixed">
+        <parent link="chassis"/>
+        <child link="fr_left_us_frame"/>
+        <origin xyz="${us_offset_x - 0.023} ${us_offset_y} ${us_offset_z}" rpy="0 0 ${us_rotation_yaw}"/>
+    </joint>
+    <link name="fr_left_us_frame">
+        <visual>
+            <geometry>
+                <box size="0.005 0.04 0.02"/>
+            </geometry>
+            <origin xyz="0 0 -0.0025" rpy="0 0 0"/>
+        </visual>
+        <collision>
+            <geometry>
+                <box size="0.005 0.04 0.02"/>
+            </geometry>
+            <origin xyz="0 0 -0.0025" rpy="0 0 0"/>
+        </collision>
+        <xacro:inertial_cylinder mass="0.1" length="0.02" radius="0.01">
+            <origin xyz="0 0 0" rpy="0 0 0"/>
+        </xacro:inertial_cylinder>
+    </link>
+    <gazebo reference="fr_left_us_frame">
+        <material>Gazebo/Red</material>
+        <sensor type="ray" name="fr_left_range_sensor">
             <visualize>true</visualize>
             <pose> 0 0 0 0 0 0 </pose>
@@ -37,13 +100,64 @@
                         <max_angle>0.087</max_angle>
                     </horizontal>
-                    <!-- <vertical>
+                </scan>
+                <range>
+                    <min>0.2</min>
+                    <max>5.0</max>
+                    <resolution>0.01</resolution>
+                </range>
+                <noise>
+                    <type>gaussian</type>
+                    <mean>0.0</mean>
+                    <stddev>0.01</stddev>
+                </noise>
+            </ray>
+            <update_rate>30</update_rate>
+            <plugin name="fr_left_us_controller" filename="libgazebo_ros_ray_sensor.so">
+                <ros>
+                    <remapping>~/out:=fr_left_range</remapping>
+                </ros>
+                <output_type>sensor_msgs/Range</output_type>
+                <frame_name>fr_left_us_frame</frame_name>
+            </plugin>
+        </sensor>
+    </gazebo>
+    <joint name="fr_right_us_joint" type="fixed">
+        <parent link="chassis"/>
+        <child link="fr_right_us_frame"/>
+        <origin xyz="${us_offset_x - 0.023} ${-us_offset_y} ${us_offset_z}" rpy="0 0 ${-us_rotation_yaw}"/>
+    </joint>
+    <link name="fr_right_us_frame">
+        <visual>
+            <geometry>
+                <box size="0.005 0.04 0.02"/>
+            </geometry>
+            <origin xyz="0 0 -0.0025" rpy="0 0 0"/>
+        </visual>
+        <collision>
+            <geometry>
+                <box size="0.005 0.04 0.02"/>
+            </geometry>
+            <origin xyz="0 0 -0.0025" rpy="0 0 0"/>
+        </collision>
+        <xacro:inertial_cylinder mass="0.1" length="0.02" radius="0.01">
+            <origin xyz="0 0 0" rpy="0 0 0"/>
+        </xacro:inertial_cylinder>
+    </link>
+    <gazebo reference="fr_right_us_frame">
+        <material>Gazebo/Red</material>
+        <sensor type="ray" name="fr_right_range_sensor">
+            <visualize>true</visualize>
+            <pose> 0 0 0 0 0 0 </pose>
+            <ray>
+                <scan>
+                    <horizontal>
                         <samples>10</samples>
                         <resolution>1</resolution>
                         <min_angle>-0.087</min_angle>
                         <max_angle>0.087</max_angle>
-                    </vertical> -->
-                </scan>
-                <range>
-                    <min>0.10</min>
+                    </horizontal>
+                </scan>
+                <range>
+                    <min>0.2</min>
                     <max>5.0</max>
                     <resolution>0.01</resolution>
@@ -54,12 +168,82 @@
                     <stddev>0.01</stddev>
                 </noise>
+                 <noise>
+                    <type>gaussian</type>
+                    <mean>0.0</mean>
+                    <stddev>0.01</stddev>
+                </noise>
             </ray>
             <update_rate>30</update_rate>
-            <plugin name="gazebo_ros_range_controller" filename="libgazebo_ros_ray_sensor.so">
-                <ros>
-                    <remapping>~/out:=range</remapping>
-                </ros>
-                <output_type>sensor_msgs/Range</output_type>
-                <frame_name>ultrasonic_frame</frame_name>
+            <plugin name="fr_right_us_controller" filename="libgazebo_ros_ray_sensor.so">
+                <ros>
+                    <remapping>~/out:=fr_right_range</remapping>
+                </ros>
+                <output_type>sensor_msgs/Range</output_type>
+                <frame_name>fr_right_us_frame</frame_name>
+            </plugin>
+        </sensor>
+    </gazebo> -->
+    <joint name="bc_mid_us_joint" type="fixed">
+        <parent link="chassis"/>
+        <child link="bc_mid_us_frame"/>
+        <origin xyz="${-us_offset_x} 0 ${us_offset_z}" rpy="0 0 3.14"/>
+    </joint>
+    <link name="bc_mid_us_frame">
+        <visual>
+            <geometry>
+                <box size="0.005 0.04 0.02"/>
+            </geometry>
+            <origin xyz="0 0 -0.0025" rpy="0 0 3.14"/>
+        </visual>
+        <collision>
+            <geometry>
+                <box size="0.005 0.04 0.02"/>
+            </geometry>
+            <origin xyz="0 0 -0.0025" rpy="0 0 3.14"/>
+        </collision>
+        <xacro:inertial_cylinder mass="0.1" length="0.02" radius="0.01">
+            <origin xyz="0 0 0" rpy="0 0 3.14"/>
+        </xacro:inertial_cylinder>
+    </link>
+    <gazebo reference="bc_mid_us_frame">
+        <material>Gazebo/Red</material>
+        <sensor type="ray" name="bc_mid_range_sensor">
+            <visualize>true</visualize>
+            <pose> 0 0 0 0 0 0 </pose>
+            <ray>
+                <scan>
+                    <horizontal>
+                        <samples>10</samples>
+                        <resolution>1.00000</resolution>
+                        <min_angle>-0.12</min_angle>
+                        <max_angle>0.12</max_angle>
+                    </horizontal>
+                    <vertical>
+                        <samples>5</samples>
+                        <resolution>1.00000</resolution>
+                        <min_angle>-0.01</min_angle>
+                        <max_angle>0.01</max_angle>
+                    </vertical>
+                </scan>
+                <range>
+                    <min>0.2</min>
+                    <max>5.0</max>
+                    <resolution>0.01</resolution>
+                </range>
+                 <noise>
+                    <type>gaussian</type>
+                    <mean>0.0</mean>
+                    <stddev>0.01</stddev>
+                </noise>
+            </ray>
+            <update_rate>20</update_rate>
+            <plugin name="bc_mid_us_controller" filename="libgazebo_ros_ray_sensor.so">
+                <ros>
+                    <remapping>~/out:=bc_mid_range</remapping>
+                </ros>
+                <output_type>sensor_msgs/Range</output_type>
+                <frame_name>bc_mid_us_frame</frame_name>
+                <field_of_view>0.01</field_of_view>
+                <radiation_type>ultrasound</radiation_type>
             </plugin>
         </sensor>

Commit message: update

File: description/gazebo_control.xacro (robot description, xacro)
@@ -6,6 +6,6 @@
             <left_joint>left_wheel_joint</left_joint>
             <right_joint>right_wheel_joint</right_joint>
-            <wheel_separation>0.35</wheel_separation>
-            <wheel_diameter>0.125</wheel_diameter>
+            <wheel_separation>0.29</wheel_separation>
+            <wheel_radius>0.0685</wheel_radius>
             <!-- Limits -->
             <max_wheel_torque>1</max_wheel_torque>
@@ -18,9 +18,9 @@
             <publish_wheel_tf>true</publish_wheel_tf>
         </plugin>
-        <plugin name="joint_state_publisher" filename="libgazebo_ros_joint_state_publisher.so">
+        <!-- <plugin name="joint_state_publisher" filename="libgazebo_ros_joint_state_publisher.so">
             <topic>joint_states</topic>
             <joint_name>left_wheel_joint</joint_name>
             <joint_name>right_wheel_joint</joint_name>
-        </plugin>
+        </plugin> -->
     </gazebo>
 </robot>

File: description/robot_core.xacro (robot description, xacro)
@@ -5,14 +5,14 @@
     <xacro:property name="chassis_height" value="0.2"/>
     <xacro:property name="chassis_mass" value="20.0"/>
-    <xacro:property name="wheel_radius" value="0.125"/>
-    <xacro:property name="wheel_thickness" value="0.04"/>
+    <xacro:property name="wheel_radius" value="0.0685"/>
+    <xacro:property name="wheel_thickness" value="0.037"/>
     <xacro:property name="wheel_mass" value="0.05"/>
     <xacro:property name="wheel_offset_x" value="0"/>
     <xacro:property name="wheel_offset_y" value="0.1485"/>
-    <xacro:property name="wheel_offset_z" value="0.01"/>
+    <xacro:property name="wheel_offset_z" value="0.01"/>.
     <xacro:property name="caster_wheel_radius" value="0.02"/>
     <xacro:property name="caster_wheel_mass" value="0.01"/>
     <xacro:property name="connector_size" value="0.02"/>
-    <xacro:property name="connector_height" value="0.15"/>
+    <xacro:property name="connector_height" value="0.075"/>
     <xacro:property name="connector_offset_z" value="-0.02"/>
     <xacro:property name="caster_wheel_offset_x" value="0.1"/>
