Commit message: update real robot

File: description/robot_core.xacro (robot description, xacro)
@@ -3,5 +3,5 @@
     <xacro:include filename="inertial_macros.xacro"/>
     <xacro:property name="chassis_length" value="0.44"/>
-    <xacro:property name="chassis_height" value="0.2"/>
+    <xacro:property name="chassis_height" value="1"/>
     <xacro:property name="chassis_mass" value="2.0"/>
     <xacro:property name="wheel_radius" value="0.075"/>

File: description/ros2_control.xacro (robot description, xacro)
@@ -11,5 +11,5 @@
                 <param name="baud_rate">57600</param>
                 <param name="timeout_ms">1000</param>
-                <param name="enc_counts_per_rev">28407</param>
+                <param name="enc_counts_per_rev">27850</param>
             </hardware>
             <joint name="left_wheel_joint">

Commit message: update

File: description/robot_core.xacro (robot description, xacro)
@@ -3,5 +3,5 @@
     <xacro:include filename="inertial_macros.xacro"/>
     <xacro:property name="chassis_length" value="0.44"/>
-    <xacro:property name="chassis_height" value="1"/>
+    <xacro:property name="chassis_height" value="0.2"/>
     <xacro:property name="chassis_mass" value="2.0"/>
     <xacro:property name="wheel_radius" value="0.075"/>

File: description/ros2_control.xacro (robot description, xacro)
@@ -11,5 +11,5 @@
                 <param name="baud_rate">57600</param>
                 <param name="timeout_ms">1000</param>
-                <param name="enc_counts_per_rev">27850</param>
+                <param name="enc_counts_per_rev">28407</param>
             </hardware>
             <joint name="left_wheel_joint">

Commit message: Update control

File: description/robot_core.xacro (robot description, xacro)
@@ -4,6 +4,6 @@
     <xacro:property name="chassis_length" value="0.44"/>
     <xacro:property name="chassis_height" value="0.2"/>
-    <xacro:property name="chassis_mass" value="2.0"/>
-    <xacro:property name="wheel_radius" value="0.075"/>
+    <xacro:property name="chassis_mass" value="20.0"/>
+    <xacro:property name="wheel_radius" value="0.125"/>
     <xacro:property name="wheel_thickness" value="0.05"/>
     <xacro:property name="wheel_mass" value="0.05"/>

Commit message: update size of wheels

File: description/robot_core.xacro (robot description, xacro)
@@ -5,5 +5,5 @@
     <xacro:property name="chassis_height" value="0.2"/>
     <xacro:property name="chassis_mass" value="20.0"/>
-    <xacro:property name="wheel_radius" value="0.0685"/>
+    <xacro:property name="wheel_radius" value="0.07"/>
     <xacro:property name="wheel_thickness" value="0.037"/>
     <xacro:property name="wheel_mass" value="0.05"/>
